File: KiCAD/Mixer/ch_fader.kicad_sch (KiCad schematic)
At the start: 4 parts, among them U4 NE5532

Commit message: Final PCB Version that got ordered from JLCPCB
Parts:
- RV2: value R_Potentiometer -> 10k
- renumbered R15 to R14, U4 to U2
Changed lines of the file:
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@@
 			)
 		)
-		(property "Value" "R_Potentiometer"
+		(property "Value" "10k"
 			(at 78.74 49.53 90)
 			(show_name no)
@@
 		(dnp no)
 		(fields_autoplaced yes)
-		(property "Reference" "U4"
+		(property "Reference" "U2"
 			(at 78.74 54.61 0)
 			(show_name no)
@@
 			(project "Mixer"
 				(path "/322d427a-6aae-4762-92d6-d97688daf29b/8a2849b7-184d-4014-bb98-da9dec8b5f90/e455183a-ba3c-419d-9cae-765ff61c6b78"
-					(reference "U4")
+					(reference "U2")
 					(unit 1)
 				)
@@
 		(in_pos_files yes)
 		(dnp no)
-		(property "Reference" "R15"
+		(property "Reference" "R14"
 			(at 92.202 67.31 90)
 			(show_name no)
@@
 			(project "Mixer"
 				(path "/322d427a-6aae-4762-92d6-d97688daf29b/8a2849b7-184d-4014-bb98-da9dec8b5f90/e455183a-ba3c-419d-9cae-765ff61c6b78"
-					(reference "R15")
+					(reference "R14")
 					(unit 1)
 				)
