File: KiCAD/Mixer/ch_mute.kicad_sch (KiCad schematic)
At the start: 8 parts, among them Q1 MMBFJ111, Q2 MMBFJ111, SW1 SW_MEC_5G

Commit message: Power Bus, Footprints, Audio Bus
Parts:
- R5, R6, R7, R8: footprint (none) -> Resistor_SMD:R_0805_2012Metric_Pad1.20x1.40mm_HandSolder
Changed lines of the file:
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@@
 			)
 		)
-		(property "Footprint" ""
+		(property "Footprint" "Resistor_SMD:R_0805_2012Metric_Pad1.20x1.40mm_HandSolder"
 			(at 121.92 64.008 90)
 			(hide yes)
@@
 			)
 		)
-		(property "Footprint" ""
+		(property "Footprint" "Resistor_SMD:R_0805_2012Metric_Pad1.20x1.40mm_HandSolder"
 			(at 72.39 72.898 90)
 			(hide yes)
@@
 			)
 		)
-		(property "Footprint" ""
+		(property "Footprint" "Resistor_SMD:R_0805_2012Metric_Pad1.20x1.40mm_HandSolder"
 			(at 72.39 64.008 90)
 			(hide yes)
@@
 			)
 		)
-		(property "Footprint" ""
+		(property "Footprint" "Resistor_SMD:R_0805_2012Metric_Pad1.20x1.40mm_HandSolder"
 			(at 61.468 77.47 90)
 			(hide yes)

Commit message: added second channel and footprints / created PCB desing...might make PCB bit bigger
Parts:
- C4: footprint (none) -> Capacitor_SMD:C_0805_2012Metric_Pad1.18x1.45mm_HandSolder
- SW1: footprint (none) -> Eigene:Switch BHT
Changed lines of the file:
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@@
 			)
 		)
-		(property "Footprint" ""
+		(property "Footprint" "Eigene:Switch BHT"
 			(at 49.53 66.04 0)
 			(hide yes)
@@
 					(unit 1)
 				)
+				(path "/322d427a-6aae-4762-92d6-d97688daf29b/8a2849b7-184d-4014-bb98-da9dec8b5f90/ec4e71c2-26db-4ba4-aad5-0bfc40b10850"
+					(reference "SW2")
+					(unit 1)
+				)
 			)
 		)
@@
 					(unit 1)
 				)
+				(path "/322d427a-6aae-4762-92d6-d97688daf29b/8a2849b7-184d-4014-bb98-da9dec8b5f90/ec4e71c2-26db-4ba4-aad5-0bfc40b10850"
+					(reference "R19")
+					(unit 1)
+				)
 			)
 		)
@@
 					(unit 1)
 				)
+				(path "/322d427a-6aae-4762-92d6-d97688daf29b/8a2849b7-184d-4014-bb98-da9dec8b5f90/ec4e71c2-26db-4ba4-aad5-0bfc40b10850"
+					(reference "Q4")
+					(unit 1)
+				)
 			)
 		)
@@
 					(unit 1)
 				)
+				(path "/322d427a-6aae-4762-92d6-d97688daf29b/8a2849b7-184d-4014-bb98-da9dec8b5f90/ec4e71c2-26db-4ba4-aad5-0bfc40b10850"
+					(reference "#PWR081")
+					(unit 1)
+				)
 			)
 		)
@@
 					(unit 1)
 				)
+				(path "/322d427a-6aae-4762-92d6-d97688daf29b/8a2849b7-184d-4014-bb98-da9dec8b5f90/ec4e71c2-26db-4ba4-aad5-0bfc40b10850"
+					(reference "R18")
+					(unit 1)
+				)
 			)
 		)
@@
 					(unit 1)
 				)
+				(path "/322d427a-6aae-4762-92d6-d97688daf29b/8a2849b7-184d-4014-bb98-da9dec8b5f90/ec4e71c2-26db-4ba4-aad5-0bfc40b10850"
+					(reference "#PWR085")
+					(unit 1)
+				)
 			)
 		)
@@
 					(unit 1)
 				)
+				(path "/322d427a-6aae-4762-92d6-d97688daf29b/8a2849b7-184d-4014-bb98-da9dec8b5f90/ec4e71c2-26db-4ba4-aad5-0bfc40b10850"
+					(reference "#PWR084")
+					(unit 1)
+				)
 			)
 		)
@@
 					(unit 1)
 				)
+				(path "/322d427a-6aae-4762-92d6-d97688daf29b/8a2849b7-184d-4014-bb98-da9dec8b5f90/ec4e71c2-26db-4ba4-aad5-0bfc40b10850"
+					(reference "#PWR082")
+					(unit 1)
+				)
 			)
 		)
@@
 			)
 		)
-		(property "Footprint" ""
+		(property "Footprint" "Capacitor_SMD:C_0805_2012Metric_Pad1.18x1.45mm_HandSolder"
 			(at 78.4352 87.63 0)
 			(hide yes)
@@
 					(unit 1)
 				)
+				(path "/322d427a-6aae-4762-92d6-d97688daf29b/8a2849b7-184d-4014-bb98-da9dec8b5f90/ec4e71c2-26db-4ba4-aad5-0bfc40b10850"
+					(reference "C6")
+					(unit 1)
+				)
 			)
 		)
@@
 					(unit 1)
 				)
+				(path "/322d427a-6aae-4762-92d6-d97688daf29b/8a2849b7-184d-4014-bb98-da9dec8b5f90/ec4e71c2-26db-4ba4-aad5-0bfc40b10850"
+					(reference "#PWR086")
+					(unit 1)
+				)
 			)
 		)
@@
 					(unit 1)
 				)
+				(path "/322d427a-6aae-4762-92d6-d97688daf29b/8a2849b7-184d-4014-bb98-da9dec8b5f90/ec4e71c2-26db-4ba4-aad5-0bfc40b10850"
+					(reference "Q3")
+					(unit 1)
+				)
 			)
 		)
@@
 					(unit 1)
 				)
+				(path "/322d427a-6aae-4762-92d6-d97688daf29b/8a2849b7-184d-4014-bb98-da9dec8b5f90/ec4e71c2-26db-4ba4-aad5-0bfc40b10850"
+					(reference "R17")
+					(unit 1)
+				)
 			)
 		)
@@
 					(unit 1)
 				)
+				(path "/322d427a-6aae-4762-92d6-d97688daf29b/8a2849b7-184d-4014-bb98-da9dec8b5f90/ec4e71c2-26db-4ba4-aad5-0bfc40b10850"
+					(reference "#PWR087")
+					(unit 1)
+				)
 			)
 		)
@@
 					(unit 1)
 				)
+				(path "/322d427a-6aae-4762-92d6-d97688daf29b/8a2849b7-184d-4014-bb98-da9dec8b5f90/ec4e71c2-26db-4ba4-aad5-0bfc40b10850"
+					(reference "#PWR083")
+					(unit 1)
+				)
 			)
 		)
@@
 					(unit 1)
 				)
+				(path "/322d427a-6aae-4762-92d6-d97688daf29b/8a2849b7-184d-4014-bb98-da9dec8b5f90/ec4e71c2-26db-4ba4-aad5-0bfc40b10850"
+					(reference "R16")
+					(unit 1)
+				)

Commit message: Cs an OPV-Strom, Anpassung clicklessmute,...
Parts:
- C4: value 100n -> 220n
Changed lines of the file:
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@@
 			)
 		)
-		(property "Value" "100n"
+		(property "Value" "220n"
 			(at 80.01 85.09 0)
 			(show_name no)
