File: KiCAD/Mixer/ch_mute.kicad_sch (KiCad schematic)
At the start: 9 parts, among them Q2 MMBFJ111, Q3 MMBFJ111, SW1 SW_MEC_5G

Commit message: Final PCB Version that got ordered from JLCPCB
Parts:
- renumbered C18 to C2
Changed lines of the file:
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@@
 		(in_pos_files yes)
 		(dnp no)
-		(property "Reference" "C18"
+		(property "Reference" "C2"
 			(at 69.85 82.55 0)
 			(show_name no)
@@
 			(project "Mixer"
 				(path "/322d427a-6aae-4762-92d6-d97688daf29b/8a2849b7-184d-4014-bb98-da9dec8b5f90/bf84a5ed-2042-40b8-aca0-adb831118b62"
-					(reference "C18")
+					(reference "C2")
 					(unit 1)
 				)
