File: KiCAD/Mixer/Mixer.kicad_pcb (KiCad board)
At the start: 2 copper layers, 30 x 118.5 mm, 63 parts, among them J1 AudioJack2, J2 Conn_02x05_Odd_Even, J3 Conn_02x03_Odd_Even, J4 Conn_02x08_Odd_Even, J5 AudioJack2, Q1 MMBFJ111, Q2 MMBFJ111, Q3 MMBFJ111, Q4 MMBFJ111, SW1 SW_MEC_5G, SW2 SW_MEC_5G, U1 NE5532, U2 NE5532, U3 NE5532, U4 NE5532, U5 NE5532, U6 NE5532

Commit message: Main Modul Schaltung
Parts:
- removed C1, C3: 470u, Capacitor_SMD:C_0805_2012Metric_Pad1.18x1.45mm_HandSolder
- removed C10, C4, C6, C7, C8, C9: 100n, Capacitor_SMD:C_0805_2012Metric_Pad1.18x1.45mm_HandSolder
- removed D1, D2, D5, D6: D, Diode_SMD:D_SOD-123
- removed J1, J5: AudioJack2, Connector_Audio:Jack_3.5mm_QingPu_WQP-PJ398SM_Vertical_CircularHoles
- removed J2: Conn_02x05_Odd_Even, Connector_PinHeader_2.54mm:PinHeader_2x05_P2.54mm_Vertical
- removed J3: Conn_02x03_Odd_Even, Connector_PinHeader_2.54mm:PinHeader_2x03_P2.54mm_Vertical
- removed J4: Conn_02x08_Odd_Even, Connector_PinHeader_2.54mm:PinHeader_2x08_P2.54mm_Vertical
- removed Q1, Q2, Q3, Q4: MMBFJ111, Package_TO_SOT_SMD:SOT-23
- removed R1, R10, R13, R14, R15, R2, R21, R22, R3, R9: R, Resistor_SMD:R_0805_2012Metric_Pad1.20x1.40mm_HandSolder
- removed R11, R12, R23, R24: 100, Resistor_SMD:R_0805_2012Metric_Pad1.20x1.40mm_HandSolder
- removed R16, R8: 10k, Resistor_SMD:R_0805_2012Metric_Pad1.20x1.40mm_HandSolder
- removed R17, R19, R5, R6: 2k2, Resistor_SMD:R_0805_2012Metric_Pad1.20x1.40mm_HandSolder
- removed R18, R7: 100k, Resistor_SMD:R_0805_2012Metric_Pad1.20x1.40mm_HandSolder
- removed R20, R4: 1k, Resistor_SMD:R_0805_2012Metric_Pad1.20x1.40mm_HandSolder
- removed RV1, RV5: 10k, Potentiometer_THT:Potentiometer_Alps_RK09K_Single_Vertical
- removed RV2, RV6: 1k, Potentiometer_THT:Potentiometer_Bourns_PTA1543_Single_Slide
- removed RV3, RV7: 10k, Potentiometer_THT:Potentiometer_Alps_RK09L_Double_Vertical
- removed RV4, RV8: 100, Potentiometer_THT:Potentiometer_Alps_RK09K_Single_Vertical
- removed SW1, SW2: SW_MEC_5G, Eigene:Switch BHT
- removed U1, U2, U3, U4, U5, U6: NE5532, Package_SO:SOIC-8_3.9x4.9mm_P1.27mm
- added C26: 100n, Capacitor_SMD:C_0805_2012Metric_Pad1.18x1.45mm_HandSolder, B.Cu at (143.5, 81.5)
- added C27: 100n, Capacitor_SMD:C_0805_2012Metric_Pad1.18x1.45mm_HandSolder, B.Cu at (143.5, 84.5)
- added C28: 100n, Capacitor_SMD:C_0805_2012Metric_Pad1.18x1.45mm_HandSolder, B.Cu at (188.4, 81.5)
- added C29: 100n, Capacitor_SMD:C_0805_2012Metric_Pad1.18x1.45mm_HandSolder, B.Cu at (158.3, 98.9)
- added C30: 100n, Capacitor_SMD:C_0805_2012Metric_Pad1.18x1.45mm_HandSolder, B.Cu at (158.3, 102.0)
- added C44: 100n, Capacitor_SMD:C_0805_2012Metric_Pad1.18x1.45mm_HandSolder, B.Cu at (188.4, 84.5)
- added C45: 100u, Capacitor_SMD:C_0805_2012Metric_Pad1.18x1.45mm_HandSolder, B.Cu at (188.4, 87.5)
- added C46: 390p, Capacitor_SMD:C_0805_2012Metric_Pad1.18x1.45mm_HandSolder, B.Cu at (188.4, 90.5)
- added C47: 100n, Capacitor_SMD:C_0805_2012Metric_Pad1.18x1.45mm_HandSolder, B.Cu at (143.5, 87.5)
- added C48: 100n, Capacitor_SMD:C_0805_2012Metric_Pad1.18x1.45mm_HandSolder, B.Cu at (143.5, 90.5)
- added C49: 100u, Capacitor_SMD:C_0805_2012Metric_Pad1.18x1.45mm_HandSolder, B.Cu at (188.4, 93.5)
- added C50: 390p, Capacitor_SMD:C_0805_2012Metric_Pad1.18x1.45mm_HandSolder, B.Cu at (183.6, 81.5)
- added C51: 470u, Capacitor_SMD:C_0805_2012Metric_Pad1.18x1.45mm_HandSolder, B.Cu at (217.0, 73.5)
- added C52: 470u, Capacitor_SMD:C_0805_2012Metric_Pad1.18x1.45mm_HandSolder, B.Cu at (217.0, 76.5)
- added C53: 100u, Capacitor_SMD:C_0805_2012Metric_Pad1.18x1.45mm_HandSolder, B.Cu at (183.6, 84.5)
- added C54: 100u, Capacitor_SMD:C_0805_2012Metric_Pad1.18x1.45mm_HandSolder, B.Cu at (183.6, 87.5)
- added C55: 100n, Capacitor_SMD:C_0805_2012Metric_Pad1.18x1.45mm_HandSolder, B.Cu at (183.6, 90.5)
- added C56: 100n, Capacitor_SMD:C_0805_2012Metric_Pad1.18x1.45mm_HandSolder, B.Cu at (183.6, 93.5)
- added D7: 1N5711, Diode_SMD:D_SOD-323_HandSoldering, B.Cu at (149.2, 111.2)
- added D8: 1N5711, Diode_SMD:D_SOD-323_HandSoldering, B.Cu at (152.3, 117.5)
- added J10: Send_B_L, Connector_Audio:Jack_3.5mm_QingPu_WQP-PJ398SM_Vertical_CircularHoles, F.Cu at (105.0, 65.8)
- added J11: Send_B_R, Connector_Audio:Jack_3.5mm_QingPu_WQP-PJ398SM_Vertical_CircularHoles, F.Cu at (115.0, 65.8)
- added J12: Return_A_L, Connector_Audio:Jack_3.5mm_QingPu_WQP-PJ398SM_Vertical_CircularHoles, F.Cu at (105.0, 80.2)
- added J13: Return_A_R, Connector_Audio:Jack_3.5mm_QingPu_WQP-PJ398SM_Vertical_CircularHoles, F.Cu at (115.0, 80.2)
- added J14: Return_B_L, Connector_Audio:Jack_3.5mm_QingPu_WQP-PJ398SM_Vertical_CircularHoles, F.Cu at (105.0, 94.6)
- added J15: Return_B_R, Connector_Audio:Jack_3.5mm_QingPu_WQP-PJ398SM_Vertical_CircularHoles, F.Cu at (115.0, 94.6)
- added J16: Balanced_Out_L, Connector_Audio:Jack_6.35mm_Neutrik_NJ3FD-V_Vertical, F.Cu at (115.3, 146.7)
- added J17: HPO, Connector_Audio:Jack_3.5mm_QingPu_WQP-PJ398SM_Vertical_CircularHoles, F.Cu at (105.0, 109.0)
- added J18: Balanced_Out_R, Connector_Audio:Jack_6.35mm_Neutrik_NJ3FD-V_Vertical, F.Cu at (115.3, 162.2)
- added J19: Conn_02x05_Odd_Even, Connector_IDC:IDC-Header_2x04_P2.54mm_Vertical, B.Cu at (144.2, 120.9)
- added J7: Conn_02x09_Odd_Even, Connector_PinHeader_2.54mm:PinHeader_2x09_P2.54mm_Vertical, B.Cu at (160.0, 137.4)
- added J8: Send_A_L, Connector_Audio:Jack_3.5mm_QingPu_WQP-PJ398SM_Vertical_CircularHoles, F.Cu at (105.0, 51.4)
- added J9: SendA_R, Connector_Audio:Jack_3.5mm_QingPu_WQP-PJ398SM_Vertical_CircularHoles, F.Cu at (125.0, 63.0)
- added R29: 470, Resistor_SMD:R_0805_2012Metric_Pad1.20x1.40mm_HandSolder, B.Cu at (163.1, 98.9)
- added R30: 1k, Resistor_SMD:R_0805_2012Metric_Pad1.20x1.40mm_HandSolder, B.Cu at (163.1, 101.9)
- added R31: 1k, Resistor_SMD:R_0805_2012Metric_Pad1.20x1.40mm_HandSolder, B.Cu at (163.1, 104.8)
- added R32: 1k, Resistor_SMD:R_0805_2012Metric_Pad1.20x1.40mm_HandSolder, B.Cu at (163.1, 107.8)
- added R33: 1k, Resistor_SMD:R_0805_2012Metric_Pad1.20x1.40mm_HandSolder, B.Cu at (163.1, 110.7)
- added R34: 1k, Resistor_SMD:R_0805_2012Metric_Pad1.20x1.40mm_HandSolder, B.Cu at (163.1, 113.7)
- added R35: 1k, Resistor_SMD:R_0805_2012Metric_Pad1.20x1.40mm_HandSolder, B.Cu at (163.1, 116.6)
- added R39: 10k, Resistor_SMD:R_0805_2012Metric_Pad1.20x1.40mm_HandSolder, B.Cu at (212.2, 67.4)
- added R40: 10k, Resistor_SMD:R_0805_2012Metric_Pad1.20x1.40mm_HandSolder, B.Cu at (212.2, 70.4)
- added R41: 10k, Resistor_SMD:R_0805_2012Metric_Pad1.20x1.40mm_HandSolder, B.Cu at (212.2, 73.3)
- added R42: 10k, Resistor_SMD:R_0805_2012Metric_Pad1.20x1.40mm_HandSolder, B.Cu at (212.2, 76.3)
- added R49: 22k, Resistor_SMD:R_0805_2012Metric_Pad1.20x1.40mm_HandSolder, B.Cu at (188.4, 96.5)
- added R50: 68, Resistor_SMD:R_0805_2012Metric_Pad1.20x1.40mm_HandSolder, B.Cu at (188.4, 99.5)
- added R51: 1k, Resistor_SMD:R_0805_2012Metric_Pad1.20x1.40mm_HandSolder, B.Cu at (188.4, 102.4)
- added R52: 1k, Resistor_SMD:R_0805_2012Metric_Pad1.20x1.40mm_HandSolder, B.Cu at (188.4, 105.4)
- added R53: 22k, Resistor_SMD:R_0805_2012Metric_Pad1.20x1.40mm_HandSolder, B.Cu at (183.7, 96.5)
- added R54: 68, Resistor_SMD:R_0805_2012Metric_Pad1.20x1.40mm_HandSolder, B.Cu at (183.7, 99.5)
- added R55: 1k, Resistor_SMD:R_0805_2012Metric_Pad1.20x1.40mm_HandSolder, B.Cu at (183.7, 102.4)
- added R56: 1k, Resistor_SMD:R_0805_2012Metric_Pad1.20x1.40mm_HandSolder, B.Cu at (183.7, 105.4)
- added R57: 22k, Resistor_SMD:R_0805_2012Metric_Pad1.20x1.40mm_HandSolder, B.Cu at (178.9, 96.5)
- added R58: 68, Resistor_SMD:R_0805_2012Metric_Pad1.20x1.40mm_HandSolder, B.Cu at (178.9, 99.5)
- added R59: 22k, Resistor_SMD:R_0805_2012Metric_Pad1.20x1.40mm_HandSolder, B.Cu at (178.9, 102.4)
- added R60: 68, Resistor_SMD:R_0805_2012Metric_Pad1.20x1.40mm_HandSolder, B.Cu at (178.9, 105.4)
- added R61: 470, Resistor_SMD:R_0805_2012Metric_Pad1.20x1.40mm_HandSolder, B.Cu at (163.1, 119.6)
- added R62: 1k, Resistor_SMD:R_0805_2012Metric_Pad1.20x1.40mm_HandSolder, B.Cu at (166.6, 160.6)
- added R63: 1k, Resistor_SMD:R_0805_2012Metric_Pad1.20x1.40mm_HandSolder, B.Cu at (166.6, 163.6)
- added R64: 1k, Resistor_SMD:R_0805_2012Metric_Pad1.20x1.40mm_HandSolder, B.Cu at (147.3, 145.6)
- added R65: 1k, Resistor_SMD:R_0805_2012Metric_Pad1.20x1.40mm_HandSolder, B.Cu at (147.3, 148.5)
- added RV12: 50k, Potentiometer_THT:Potentiometer_Alps_RK09L_Double_Vertical, F.Cu at (107.2, 137.4)
- added RV13: 50k, Potentiometer_THT:Potentiometer_Alps_RK09L_Double_Vertical, B.Cu at (167.3, 149.1)
- added U10: NE5532, Package_SO:SOIC-8_3.9x4.9mm_P1.27mm, B.Cu at (150.2, 83.3)
- added U11: NE5532, Package_SO:SOIC-8_3.9x4.9mm_P1.27mm, B.Cu at (152.4, 93.3)
- added U12: NE5532, Package_SO:SOIC-8_3.9x4.9mm_P1.27mm, B.Cu at (186.6, 110.2)
- added U13: NE5532, Package_SO:SOIC-8_3.9x4.9mm_P1.27mm, B.Cu at (186.6, 116.8)
- C2: value 100n -> 4.7u
- C5: value 100n -> 470u
- moved C2 215.6 mm to (217.0, 67.5), turned to 180 degrees
- moved C5 203.2 mm to (217.0, 70.5), turned to 180 degrees
Connections:
- C2 pad 1: GND -> Net-(C2-Pad1)
- C2 pad 2: +12V -> /Main/Send_Return/Return_A_L
- C5 pad 1: GND -> Net-(C5-Pad1)
- C5 pad 2: +12V -> /Main/Send_Return/Return_A_R
Other:
- board size 30 x 118.5 mm -> 30 x 120 mm
