File: KiCAD/Mixer/Mixer.kicad_pcb (KiCad board)
At the start: 4 copper layers, 57 x 110 mm, 145 parts, among them J1 Conn_02x09_Odd_Even, J2 Conn_02x09_Odd_Even, J3 AudioJack2, J4 Conn_01x02_Socket, J5 Conn_01x02_Socket, J6 Conn_02x05_Odd_Even, J7 Conn_01x02_Socket, J8 Conn_01x02_Socket, J9 AudioJack2, Q1 NPN, Q2 MMBFJ111, Q3 MMBFJ111, Q4 NPN, Q5 MMBFJ111, Q6 MMBFJ111, SW1 SW_MEC_5G, SW2 SW_MEC_5G, U1 NE5532, U10 NE5532, U11 NE5532, U2 NE5532, U3 NE5532, U4 NE5532, U6 NE5532, U7 NE5532, U8 NE5532, U9 NE5532

Commit message: Final PCB Version that got ordered from JLCPCB
Parts:
- removed the C10 at (75.0, 112.8)
- removed the C21 at (114.3, 40.4)
- removed the C22 at (114.8, 134.2)
- removed the C9 at (67.5, 112.8)
- removed the R53 at (92.9, 69.2)
- removed R79: 10k, Resistor_SMD:R_0805_2012Metric_Pad1.20x1.40mm_HandSolder
- removed R81, R85: 1k, Resistor_SMD:R_0805_2012Metric_Pad1.20x1.40mm_HandSolder
- removed R83, R87, R89, R91: 3k3, Resistor_SMD:R_0805_2012Metric_Pad1.20x1.40mm_HandSolder
- removed RV11: 100K, Potentiometer_THT:Potentiometer_Alps_RK09K_Single_Vertical
- removed RV12: 10k, Potentiometer_THT:Potentiometer_Alps_RK09L_Double_Vertical
- added C13: 100n, Capacitor_SMD:C_0805_2012Metric_Pad1.18x1.45mm_HandSolder, B.Cu at (67.5, 112.8)
- added C14: 100n, Capacitor_SMD:C_0805_2012Metric_Pad1.18x1.45mm_HandSolder, B.Cu at (75.0, 112.9)
- added C25: 2u, Capacitor_SMD:C_0805_2012Metric_Pad1.18x1.45mm_HandSolder, B.Cu at (114.4, 40.4)
- added C26: 220n, Capacitor_SMD:C_0805_2012Metric_Pad1.18x1.45mm_HandSolder, B.Cu at (114.8, 134.2)
- added R56: 0R, Resistor_SMD:R_0805_2012Metric_Pad1.20x1.40mm_HandSolder, F.Cu at (95.0, 72.5)
- added R58: 8k6, Resistor_SMD:R_0805_2012Metric_Pad1.20x1.40mm_HandSolder, B.Cu at (94.9, 70.0)
- added R69: 3k3, Resistor_SMD:R_0805_2012Metric_Pad1.20x1.40mm_HandSolder, B.Cu at (105.1, 107.1)
- added R70: 3k3, Resistor_SMD:R_0805_2012Metric_Pad1.20x1.40mm_HandSolder, B.Cu at (105.0, 118.4)
- added R71: 1k, Resistor_SMD:R_0805_2012Metric_Pad1.20x1.40mm_HandSolder, B.Cu at (103.1, 107.1)
- added R72: 3k3, Resistor_SMD:R_0805_2012Metric_Pad1.20x1.40mm_HandSolder, B.Cu at (107.1, 107.1)
- added R73: 3k3, Resistor_SMD:R_0805_2012Metric_Pad1.20x1.40mm_HandSolder, B.Cu at (107.0, 118.4)
- added R74: 1k, Resistor_SMD:R_0805_2012Metric_Pad1.20x1.40mm_HandSolder, B.Cu at (103.0, 118.4)
- added REF**: OSHW-Logo_5.7x6mm_SilkScreen, Symbol:OSHW-Logo_5.7x6mm_SilkScreen, B.Cu at (81.2, 33.9)
- added REF**: WEEE-Logo_4.2x6mm_SilkScreen, Symbol:WEEE-Logo_4.2x6mm_SilkScreen, B.Cu at (95.2, 34.1)
- added RV10: 10k, Potentiometer_THT:Potentiometer_Alps_RK09L_Double_Vertical, F.Cu at (106.9, 80.1)
- added RV9: 100K, Potentiometer_THT:Potentiometer_Alps_RK09K_Single_Vertical, F.Cu at (92.7, 46.8)
- D3, D4: footprint Diode_SMD:D_MiniMELF -> Diode_SMD:D_SOD-123
- R21: renamed from R19; value 1k -> 10k
- R22: renamed from R20; value 1k -> 10k
- R23: renamed from R21; value 1k -> 10k
- R24: renamed from R22; value 1k -> 10k
- R25: renamed from R23; value 1k -> 10k
- R26: renamed from R24; value 1k -> 10k
- R27: renamed from R25; value 1k -> 10k
- R28: renamed from R26; value 1k -> 10k
- R55: value 0R -> 10k
- R59: value 8k6 -> 10k
- RV2: value R_Potentiometer -> 10k
- RV4: renamed from RV5; value 1k -> 10k
- RV5: renamed from RV6; value 1k -> 10k
- RV6: renamed from RV7; value 1k -> 10k
- RV7: renamed from RV8; value 1k -> 10k
- moved R59 6.28 mm to (93.8, 72.9), turned to 0 degrees
- moved R12 3.98 mm to (68.8, 133.9)
- moved R55 3.77 mm to (93.0, 72.5)
- moved R4 3.30 mm to (83.5, 70.0)
- moved R5 3.30 mm to (81.5, 70.0)
- moved C8 3.30 mm to (88.2, 69.3)
- moved R13 3.30 mm to (81.5, 72.5)
- moved R14 3.30 mm to (83.5, 72.5)
- moved C3 3.30 mm to (88.2, 74.4)
- moved C4 3.30 mm to (88.2, 66.9)
- moved J4 3.30 mm to (76.0, 73.9)
- moved J5 3.30 mm to (76.0, 70.1)
- moved U1 3.30 mm to (88.2, 70.6)
- moved C7 3.30 mm to (88.3, 76.9)
- moved R6 3.30 mm to (82.5, 72.9)
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- renumbered C20 to C10, C7 to C11, C8 to C12, C11 to C15, C12 to C16, C13 to C17, C14 to C18, C15 to C19, C18 to C2, C16 to C20, C25 to C21, C26 to C22, C27 to C23, C28 to C24, C1 to C3, C2 to C4, C3 to C5, C4 to C6, C5 to C7, C6 to C8, C19 to C9, R15 to R14, R82 to R15, R86 to R16, R80 to R17, R90 to R18, R88 to R19, R84 to R20, R27 to R29, R28 to R30, R29 to R31, R30 to R32, R31 to R33, R32 to R34, R33 to R35, R34 to R36, R35 to R37, R36 to R38, R37 to R39, R38 to R40, R39 to R41, R40 to R42, R41 to R43, R42 to R44, R43 to R45, R44 to R46, R45 to R47, R46 to R48, R47 to R49, R6 to R5, R48 to R50, R49 to R51, R50 to R52, R51 to R53, R52 to R54, R58 to R6, RV4 to RV3, RV3 to RV8, U3 to U10, U4 to U2, U2 to U3, U8 to U4, U10 to U5, U9 to U6, U11 to U7, U6 to U8, U7 to U9
Connections:
- R55 pad 1: /Channel/Fader1/fader_out -> /Channel/Fader1/fader_in
- R55 pad 2: Net-(R55-Pad2) -> Net-(U2B--)
- R59 pad 1: Net-(U1B--) -> Net-(J7-Pin_2)
- R59 pad 2: Net-(J7-Pin_1) -> Net-(R59-Pad2)
- RV8 pad 1: Net-(R55-Pad2) -> Net-(R56-Pad2)
- RV8 pad 2: Net-(R55-Pad2) -> Net-(R56-Pad2)
- RV8 pad 3: Net-(U4B--) (its old number) -> Net-(U2B--)
- U2 pad 6: Net-(U4B--) (its old number) -> Net-(U2B--)
- U2 pad 7: Net-(R55-Pad2) -> Net-(R56-Pad2)
Routing:
- net /Channel/+12V: track 0.00 -> 281.6 mm, vias 0 -> 16
- net /Channel/-12V: track 0.00 -> 220.1 mm, vias 0 -> 10
- net GND: track 0.00 -> 119.7 mm, vias 0 -> 163
- net /Channel/pre_send2R: track 0.00 -> 86.4 mm, vias 0 -> 7
- net /Channel/Ch1_outR: track 0.00 -> 83.8 mm, vias 0 -> 5
- net /Channel/Ch2_outL: track 0.00 -> 82.3 mm, vias 0 -> 3
- net Net-(U2A--): track 0.00 -> 76.8 mm, vias 0 -> 4
- net Net-(U2B--): track 0.00 -> 74.9 mm, vias 0 -> 6
- net Net-(U5B--): track 0.00 -> 70.8 mm, vias 0 -> 1
- net /Channel/Ch2_outR: track 0.00 -> 69.2 mm, vias 0 -> 4
- net /Channel/Ch1_outL: track 0.00 -> 69.2 mm, vias 0 -> 3
- net Net-(U4B--): track 0.00 -> 68.9 mm, vias 0 -> 2
- net /Channel/Fader/fader_in: track 0.00 -> 68.1 mm, vias 0 -> 3
- net Net-(U5A--): track 0.00 -> 67.6 mm, vias 0 -> 1
- net Net-(U4A--): track 0.00 -> 65.3 mm, vias 0 -> 1
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- added copper zone on B.Cu, net GND
- added copper zone on F.Cu, net GND
- added copper zone on In1.Cu, net GND
- added copper zone on In2.Cu, net GND
Other:
- board text added: "MIXER_SYSTEM_v01.1 Channel_Module_v01.1 Designed by L. Kezele D. Born G. Harms"
