File: KiCAD/Mixer/Mixer.kicad_sch (KiCad schematic)
At the start: 0 parts

Commit message: Main Modul Schaltung
Other:
- removed sheet Channel
Changed lines of the file:
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@@
-		)
-	)
-	(sheet
-		(at 58.42 80.01)
-		(size 35.56 33.02)
-		(exclude_from_sim no)
-		(in_bom yes)
-		(on_board yes)
-		(dnp no)
-		(fields_autoplaced yes)
-		(stroke
-			(width 0.1524)
-			(type solid)
-		)
-		(fill
-			(color 0 0 0 0)
-		)
-		(property "Sheetname" "Channel"
-			(at 58.42 79.2984 0)
-			(show_name no)
-			(do_not_autoplace no)
-			(effects
-				(font
-					(size 1.27 1.27)
-				)
-				(justify left bottom)
-			)
-		)
-		(property "Sheetfile" "channel.kicad_sch"
-			(at 58.42 113.6146 0)
-			(show_name no)
-			(do_not_autoplace no)
-			(effects
-				(font
-					(size 1.27 1.27)
-				)
-				(justify left top)
-			)
-		)
-		(instances
-			(project "Mixer"
-				(path "/322d427a-6aae-4762-92d6-d97688daf29b"
-					(page "2")
-				)
-			)
 		)
 	)
