File: KiCAD/Mixer/ch_pan.kicad_sch (KiCad schematic)
At the start: 3 parts

Commit message: Main Modul Schaltung
Connections:
- net GND: now also RV3.4; no longer RV3.6
- net pan_in: now also RV3.6; no longer RV3.4
Changed lines of the file:
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@@
 		(lib_id "Device:R_Potentiometer_Dual_Separate")
 		(at 46.99 49.53 0)
+		(mirror x)
 		(unit 2)
 		(body_style 1)
@@
 		(dnp no)
 		(property "Reference" "RV3"
-			(at 45.974 48.26 0)
+			(at 45.974 50.8 0)
 			(show_name no)
 			(do_not_autoplace no)
@@
 		)
 		(property "Value" "10k"
-			(at 42.926 51.308 0)
+			(at 42.926 47.752 0)
 			(show_name no)
 			(do_not_autoplace no)
