File: KiCAD/Mixer/ch_power.kicad_sch (KiCad schematic)
At the start: 3 parts, among them J6 Conn_02x05_Odd_Even

Commit message: Main Modul Schaltung
Parts:
- D7: renamed from D3; footprint Diode_THT:D_DO-35_SOD27_P7.62mm_Horizontal -> Diode_SMD:D_SOD-323_HandSoldering
- D8: renamed from D4; footprint Diode_THT:D_DO-35_SOD27_P7.62mm_Horizontal -> Diode_SMD:D_SOD-323_HandSoldering
- J19: renamed from J6; footprint Connector_PinHeader_2.54mm:PinHeader_2x05_P2.54mm_Vertical_SMD -> Connector_IDC:IDC-Header_2x04_P2.54mm_Vertical
Other:
- note added: "ferrite beads und kondensatoren!"
Changed lines of the file:
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@@
 	(generator_version "10.0")
 	(paper "A4")
+	(text "ferrite beads  und kondensatoren!"
+		(exclude_from_sim no)
+		(at 38.1 23.622 0)
+		(effects
+			(font
+				(size 1.27 1.27)
+			)
+		)
+	)
 	(junction
 		(at 62.23 35.56)
@@
 		(dnp no)
 		(fields_autoplaced yes)
-		(property "Reference" "D3"
+		(property "Reference" "D7"
 			(at 64.77 28.8925 90)
 			(show_name no)
@@
 			)
 		)
-		(property "Footprint" "Diode_THT:D_DO-35_SOD27_P7.62mm_Horizontal"
+		(property "Footprint" "Diode_SMD:D_SOD-323_HandSoldering"
 			(at 57.785 30.48 0)
 			(hide yes)
@@
 		(instances
 			(project "Mixer"
-				(path "/322d427a-6aae-4762-92d6-d97688daf29b/8a2849b7-184d-4014-bb98-da9dec8b5f90/932feda2-710a-4894-b943-37dbe0c193d3"
-					(reference "D3")
+				(path "/322d427a-6aae-4762-92d6-d97688daf29b/2bdf0d3e-99d6-4fd9-a48e-373c3c910b53/a05199cc-8720-434a-8cee-06adcbb81d6b"
+					(reference "D7")
 					(unit 1)
 				)
@@
 		(dnp no)
 		(fields_autoplaced yes)
-		(property "Reference" "J6"
+		(property "Reference" "J19"
 			(at 62.23 36.83 0)
 			(show_name no)
@@
 			)
 		)
-		(property "Footprint" "Connector_PinHeader_2.54mm:PinHeader_2x05_P2.54mm_Vertical_SMD"
+		(property "Footprint" "Connector_IDC:IDC-Header_2x04_P2.54mm_Vertical"
 			(at 60.96 48.26 0)
 			(hide yes)
@@
 		(instances
 			(project "Mixer"
-				(path "/322d427a-6aae-4762-92d6-d97688daf29b/8a2849b7-184d-4014-bb98-da9dec8b5f90/932feda2-710a-4894-b943-37dbe0c193d3"
-					(reference "J6")
+				(path "/322d427a-6aae-4762-92d6-d97688daf29b/2bdf0d3e-99d6-4fd9-a48e-373c3c910b53/a05199cc-8720-434a-8cee-06adcbb81d6b"
+					(reference "J19")
 					(unit 1)
 				)
@@
 		(dnp no)
 		(fields_autoplaced yes)
-		(property "Reference" "D4"
+		(property "Reference" "D8"
 			(at 64.77 61.9125 90)
 			(show_name no)
@@
 			)
 		)
-		(property "Footprint" "Diode_THT:D_DO-35_SOD27_P7.62mm_Horizontal"
+		(property "Footprint" "Diode_SMD:D_SOD-323_HandSoldering"
 			(at 57.785 63.5 0)
 			(hide yes)
@@
 		(instances
 			(project "Mixer"
-				(path "/322d427a-6aae-4762-92d6-d97688daf29b/8a2849b7-184d-4014-bb98-da9dec8b5f90/932feda2-710a-4894-b943-37dbe0c193d3"
-					(reference "D4")
+				(path "/322d427a-6aae-4762-92d6-d97688daf29b/2bdf0d3e-99d6-4fd9-a48e-373c3c910b53/a05199cc-8720-434a-8cee-06adcbb81d6b"
+					(reference "D8")
 					(unit 1)
 				)
