File: KiCAD/Mixer/main.kicad_sch (KiCad schematic)
At the start: 0 parts

Commit message: Main Modul Schaltung
Other:
- removed sheet Fader
- added sheet 6.3mm_Out (6.3mm_Out.kicad_sch)
- added sheet Channel Power (ch_power.kicad_sch)
- sheet Headphone ports: added +12V, -12V, GND, Sum_In_L, Sum_In_R; removed none
- sheet Inputs ports: added GND, Main_Mix_L, Main_Mix_R, Send_A_L, Send_A_R, Send_B_L, Send_B_R; removed none
- sheet Send_Return ports: added GND, Return_A_L, Return_A_R, Return_B_L, Return_B_R, Send_A_L, Send_A_R, Send_B_L, Send_B_R; removed none
- sheet Sum ports: added +12V, -12V, GND, Main_Mix_L, Main_Mix_R, Return_A_L, Return_A_R, Return_B_L, Return_B_R, Sum_Out_L, Sum_Out_R; removed none
- note added: "Balanced Out, Headphone Amp, Gain, 9 Pin in put, Metering/LEDs, Runde Abstände der Bauteile, 4 layer PCB"
