File: KiCAD/Mixer/main_fader.kicad_sch (KiCad schematic)
At the start: 0 parts

Commit message: Main Modul Schaltung
Parts:
- added R36, R37, R38: R, Resistor_SMD:R_0805_2012Metric_Pad1.20x1.40mm_HandSolder, symbol Device:R
- added RV11: 10k, Potentiometer_THT:Potentiometer_Alps_RK09K_Single_Vertical, symbol Device:R_Potentiometer
- added U9: NE5532, symbol Amplifier_Operational:NE5532
Connections:
- new net: R36.2, RV11.1
- new net: R37.1, RV11.2
- new net GND: RV11.3, U9.5 (+)
- new net gain_in: R36.1
- new net gain_out: R37.2, R38.1, R38.2, U9.6 (-), U9.7
- no-connect marks 0 -> 2
