File: KiCAD/Mixer/main_hp.kicad_sch (KiCad schematic)
At the start: 0 parts

Commit message: Main Modul Schaltung
Parts:
- added C26, C27, C47, C48: 100n, Capacitor_SMD:C_0805_2012Metric_Pad1.18x1.45mm_HandSolder, symbol Device:C
- added J17: HPO, Connector_Audio:Jack_3.5mm_QingPu_WQP-PJ398SM_Vertical_CircularHoles, symbol Connector_Audio:AudioJack3
- added R36, R37, R43, R44: 10k, symbol Device:R
- added R45, R46, R47, R48: 75, symbol Device:R
- added R64, R65: 1k, Resistor_SMD:R_0805_2012Metric_Pad1.20x1.40mm_HandSolder, symbol Device:R
- added RV12: 50k, Potentiometer_THT:Potentiometer_Alps_RK09L_Double_Vertical, symbol Device:R_Potentiometer_Dual
- added U10, U11: NE5532, Package_SO:SOIC-8_3.9x4.9mm_P1.27mm, symbol Amplifier_Operational:NE5532
Connections:
- new net: R65.2, RV12.4
- new net: R44.2, R46.1, U10.3 (+), U10.7
- new net: J17.T, R45.2, R46.2
- new net: R64.2, RV12.1
- new net: R36.2, R44.1, U10.6 (-)
- new net: R36.1, RV12.2
- new net: R37.1, RV12.5
- new net: R43.2, R48.1, U11.1, U11.5 (+)
- new net: J17.R, R47.2, R48.2
- new net: R47.1, U11.6 (-), U11.7
- new net: R37.2, R43.1, U11.2 (-)
- new net: R45.1, U10.1, U10.2 (-)
- new net +12V: C26.2, C48.2, U10.8 (V+), U11.8 (V+)
- new net -12V: C27.2, C47.2, U10.4 (V-), U11.4 (V-)
- new net GND: C26.1, C27.1, C47.1, C48.1, J17.S, RV12.3, RV12.6, U10.5 (+), U11.3 (+)
- new net Sum_In_L: R64.1
- new net Sum_In_R: R65.1
Other:
- note added: "Potentiometer/Spannungsteiler? 1k und 50 k ok? auch bei balanced out"
