File: KiCAD/Mixer/main_inputs.kicad_sch (KiCad schematic)
At the start: 0 parts

Commit message: Main Modul Schaltung
Parts:
- added J7: Conn_02x09_Odd_Even, Connector_PinHeader_2.54mm:PinHeader_2x09_P2.54mm_Vertical, symbol Connector_Generic:Conn_02x09_Odd_Even
Connections:
- new net GND: J7.13 (Pin_13), J7.14 (Pin_14), J7.3 (Pin_3), J7.4 (Pin_4), J7.7 (Pin_7), J7.8 (Pin_8)
- new net Main_Mix_L: J7.1 (Pin_1), J7.2 (Pin_2)
- new net Main_Mix_R: J7.5 (Pin_5), J7.6 (Pin_6)
- new net Send_A_L: J7.10 (Pin_10), J7.9 (Pin_9)
- new net Send_A_R: J7.11 (Pin_11), J7.12 (Pin_12)
- new net Send_B_L: J7.15 (Pin_15), J7.16 (Pin_16)
- new net Send_B_R: J7.17 (Pin_17), J7.18 (Pin_18)
