File: KiCAD/Mixer/main_send_return.kicad_sch (KiCad schematic)
At the start: 0 parts

Commit message: Main Modul Schaltung
Parts:
- added C2: 4.7u, Capacitor_SMD:C_0805_2012Metric_Pad1.18x1.45mm_HandSolder, symbol Device:C
- added C5, C51, C52: 470u, Capacitor_SMD:C_0805_2012Metric_Pad1.18x1.45mm_HandSolder, symbol Device:C
- added J10: Send_B_L, Connector_Audio:Jack_3.5mm_QingPu_WQP-PJ398SM_Vertical_CircularHoles, symbol Connector_Audio:AudioJack2
- added J11: Send_B_R, Connector_Audio:Jack_3.5mm_QingPu_WQP-PJ398SM_Vertical_CircularHoles, symbol Connector_Audio:AudioJack2
- added J12: Return_A_L, Connector_Audio:Jack_3.5mm_QingPu_WQP-PJ398SM_Vertical_CircularHoles, symbol Connector_Audio:AudioJack2
- added J13: Return_A_R, Connector_Audio:Jack_3.5mm_QingPu_WQP-PJ398SM_Vertical_CircularHoles, symbol Connector_Audio:AudioJack2
- added J14: Return_B_L, Connector_Audio:Jack_3.5mm_QingPu_WQP-PJ398SM_Vertical_CircularHoles, symbol Connector_Audio:AudioJack2
- added J15: Return_B_R, Connector_Audio:Jack_3.5mm_QingPu_WQP-PJ398SM_Vertical_CircularHoles, symbol Connector_Audio:AudioJack2
- added J8: Send_A_L, Connector_Audio:Jack_3.5mm_QingPu_WQP-PJ398SM_Vertical_CircularHoles, symbol Connector_Audio:AudioJack2
- added J9: SendA_R, Connector_Audio:Jack_3.5mm_QingPu_WQP-PJ398SM_Vertical_CircularHoles, symbol Connector_Audio:AudioJack2
- added R39, R40, R41, R42: 10k, Resistor_SMD:R_0805_2012Metric_Pad1.20x1.40mm_HandSolder, symbol Device:R
Connections:
- new net: C52.1, J15.T
- new net: C5.1, J13.T
- new net: C51.1, J14.T
- new net: C2.1, J12.T
- new net GND: J10.S, J11.S, J12.S, J13.S, J14.S, J15.S, J8.S, J9.S, R39.2, R40.2, R41.2, R42.2
- new net Return_A_L: C2.2, R39.1
- new net Return_A_R: C5.2, R40.1
- new net Return_B_L: C51.2, R41.1
- new net Return_B_R: C52.2, R42.1
- new net Send_A_L: J8.T
- new net Send_A_R: J9.T
- new net Send_B_L: J10.T
- new net Send_B_R: J11.T
Other:
- note added: "Kondensator kleiner? Pull down resistor?"
