File: KiCAD/Mixer/main_sum.kicad_sch (KiCad schematic)
At the start: 0 parts

Commit message: Main Modul Schaltung
Parts:
- added C29, C30: 100n, Capacitor_SMD:C_0805_2012Metric_Pad1.18x1.45mm_HandSolder, symbol Device:C
- added R29, R61: 470, Resistor_SMD:R_0805_2012Metric_Pad1.20x1.40mm_HandSolder, symbol Device:R
- added R30, R31, R32, R33, R34, R35: 1k, Resistor_SMD:R_0805_2012Metric_Pad1.20x1.40mm_HandSolder, symbol Device:R
- added U1: NE5532, symbol Amplifier_Operational:NE5532
Connections:
- new net: R31.2, R33.2, R35.2, R61.1, U1.6 (-)
- new net: R29.1, R30.2, R32.2, R34.2, U1.2 (-)
- new net +12V: C29.2, U1.8 (V+)
- new net -12V: C30.2, U1.4 (V-)
- new net GND: C29.1, C30.1, U1.3 (+), U1.5 (+)
- new net Main_Mix_L: R30.1
- new net Main_Mix_R: R31.1
- new net Return_A_L: R32.1
- new net Return_A_R: R33.1
- new net Return_B_L: R34.1
- new net Return_B_R: R35.1
- new net Sum_Out_L: R29.2, U1.1
- new net Sum_Out_R: R61.2, U1.7
