File: KiCAD/Mixer/ch_gain.kicad_sch (KiCad schematic)
At the start: 8 parts, among them J4 Conn_01x02_Socket, J5 Conn_01x02_Socket, U1 NE5532

Commit message: Final PCB Version that got ordered from JLCPCB
Parts:
- renumbered R6 to R5, R58 to R6
Changed lines of the file:
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@@
 		(in_pos_files yes)
 		(dnp no)
-		(property "Reference" "R6"
+		(property "Reference" "R5"
 			(at 81.788 65.532 0)
 			(show_name no)
@@
 			(project "Mixer"
 				(path "/322d427a-6aae-4762-92d6-d97688daf29b/8a2849b7-184d-4014-bb98-da9dec8b5f90/874eb9e3-c612-43fb-9dc5-24309708e7ee"
-					(reference "R6")
+					(reference "R5")
 					(unit 1)
 				)
@@
 		(in_pos_files yes)
 		(dnp no)
-		(property "Reference" "R58"
+		(property "Reference" "R6"
 			(at 100.838 66.802 90)
 			(show_name no)
@@
 			(project "Mixer"
 				(path "/322d427a-6aae-4762-92d6-d97688daf29b/8a2849b7-184d-4014-bb98-da9dec8b5f90/874eb9e3-c612-43fb-9dc5-24309708e7ee"
-					(reference "R58")
+					(reference "R6")
 					(unit 1)
 				)
