File: KiCAD/Mixer/ch_inputs.kicad_sch (KiCad schematic)
At the start: 8 parts, among them J3 AudioJack2, Q1 NPN

Commit message: Final PCB Version that got ordered from JLCPCB
Parts:
- removed C17: 2u, Capacitor_SMD:C_0805_2012Metric_Pad1.18x1.45mm_HandSolder, symbol Device:C
- added C1: 2u, Capacitor_SMD:C_0805_2012Metric_Pad1.18x1.45mm_HandSolder, symbol Device:C
Connections:
- net inputs_out: now also C1.2
- net at J3.T: now also C1.1
