File: KiCAD/Mixer/ch_main_mix.kicad_sch (KiCad schematic)
At the start: 16 parts, among them U6 NE5532, U7 NE5532

Commit message: Final PCB Version that got ordered from JLCPCB
Parts:
- renumbered R39 to R41, R40 to R42, R41 to R43, R42 to R44, R43 to R45, R44 to R46, R45 to R47, R46 to R48, R47 to R49, R48 to R50, R49 to R51, R50 to R52, R51 to R53, R52 to R54, U6 to U8, U7 to U9
Changed lines of the file:
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@@
 		(in_pos_files yes)
 		(dnp no)
-		(property "Reference" "R51"
+		(property "Reference" "R53"
 			(at 149.352 48.26 90)
 			(show_name no)
@@
 			(project "Mixer"
 				(path "/322d427a-6aae-4762-92d6-d97688daf29b/8a2849b7-184d-4014-bb98-da9dec8b5f90/2339b41c-0b4b-469c-8280-8e71cc37578f"
-					(reference "R51")
+					(reference "R53")
 					(unit 1)
 				)
@@
 		(in_pos_files yes)
 		(dnp no)
-		(property "Reference" "R50"
+		(property "Reference" "R52"
 			(at 135.89 70.104 90)
 			(show_name no)
@@
 			(project "Mixer"
 				(path "/322d427a-6aae-4762-92d6-d97688daf29b/8a2849b7-184d-4014-bb98-da9dec8b5f90/2339b41c-0b4b-469c-8280-8e71cc37578f"
-					(reference "R50")
+					(reference "R52")
 					(unit 1)
 				)
@@
 		(dnp no)
 		(fields_autoplaced yes)
-		(property "Reference" "R47"
+		(property "Reference" "R49"
 			(at 121.92 36.83 90)
 			(show_name no)
@@
 			(project "Mixer"
 				(path "/322d427a-6aae-4762-92d6-d97688daf29b/8a2849b7-184d-4014-bb98-da9dec8b5f90/2339b41c-0b4b-469c-8280-8e71cc37578f"
-					(reference "R47")
+					(reference "R49")
 					(unit 1)
 				)
@@
 		(dnp no)
 		(fields_autoplaced yes)
-		(property "Reference" "R45"
+		(property "Reference" "R47"
 			(at 99.06 26.67 90)
 			(show_name no)
@@
 			(project "Mixer"
 				(path "/322d427a-6aae-4762-92d6-d97688daf29b/8a2849b7-184d-4014-bb98-da9dec8b5f90/2339b41c-0b4b-469c-8280-8e71cc37578f"
-					(reference "R45")
+					(reference "R47")
 					(unit 1)
 				)
@@
 		(in_pos_files yes)
 		(dnp no)
-		(property "Reference" "R42"
+		(property "Reference" "R44"
 			(at 76.2 60.96 90)
 			(show_name no)
@@
 			(project "Mixer"
 				(path "/322d427a-6aae-4762-92d6-d97688daf29b/8a2849b7-184d-4014-bb98-da9dec8b5f90/2339b41c-0b4b-469c-8280-8e71cc37578f"
-					(reference "R42")
+					(reference "R44")
 					(unit 1)
 				)
@@
 		(in_pos_files yes)
 		(dnp no)
-		(property "Reference" "R43"
+		(property "Reference" "R45"
 			(at 76.2 64.77 90)
 			(show_name no)
@@
 			(project "Mixer"
 				(path "/322d427a-6aae-4762-92d6-d97688daf29b/8a2849b7-184d-4014-bb98-da9dec8b5f90/2339b41c-0b4b-469c-8280-8e71cc37578f"
-					(reference "R43")
+					(reference "R45")
 					(unit 1)
 				)
@@
 		(in_pos_files yes)
 		(dnp no)
-		(property "Reference" "R39"
+		(property "Reference" "R41"
 			(at 74.93 35.56 90)
 			(show_name no)
@@
 			(project "Mixer"
 				(path "/322d427a-6aae-4762-92d6-d97688daf29b/8a2849b7-184d-4014-bb98-da9dec8b5f90/2339b41c-0b4b-469c-8280-8e71cc37578f"
-					(reference "R39")
+					(reference "R41")
 					(unit 1)
 				)
@@
 		(dnp no)
 		(fields_autoplaced yes)
-		(property "Reference" "U7"
+		(property "Reference" "U9"
 			(at 135.89 35.56 0)
 			(show_name no)
@@
 			(project "Mixer"
 				(path "/322d427a-6aae-4762-92d6-d97688daf29b/8a2849b7-184d-4014-bb98-da9dec8b5f90/2339b41c-0b4b-469c-8280-8e71cc37578f"
-					(reference "U7")
+					(reference "U9")
 					(unit 1)
 				)
@@
 		(dnp no)
 		(fields_autoplaced yes)
-		(property "Reference" "#PWR021"
+		(property "Reference" "#PWR017"
 			(at 29.21 57.15 0)
 			(hide yes)
@@
 			(project "Mixer"
 				(path "/322d427a-6aae-4762-92d6-d97688daf29b/8a2849b7-184d-4014-bb98-da9dec8b5f90/2339b41c-0b4b-469c-8280-8e71cc37578f"
-					(reference "#PWR021")
+					(reference "#PWR017")
 					(unit 1)
 				)
@@
 		(in_pos_files yes)
 		(dnp no)
-		(property "Reference" "R44"
+		(property "Reference" "R46"
 			(at 76.2 68.58 90)
 			(show_name no)
@@
 			(project "Mixer"
 				(path "/322d427a-6aae-4762-92d6-d97688daf29b/8a2849b7-184d-4014-bb98-da9dec8b5f90/2339b41c-0b4b-469c-8280-8e71cc37578f"
-					(reference "R44")
+					(reference "R46")
 					(unit 1)
 				)
@@
 		(in_pos_files yes)
 		(dnp no)
-		(property "Reference" "R41"
+		(property "Reference" "R43"
 			(at 74.93 43.18 90)
 			(show_name no)
@@
 			(project "Mixer"
 				(path "/322d427a-6aae-4762-92d6-d97688daf29b/8a2849b7-184d-4014-bb98-da9dec8b5f90/2339b41c-0b4b-469c-8280-8e71cc37578f"
-					(reference "R41")
+					(reference "R43")
 					(unit 1)
 				)
@@
 		(in_pos_files yes)
 		(dnp no)
-		(property "Reference" "R40"
+		(property "Reference" "R42"
 			(at 74.93 39.37 90)
 			(show_name no)
@@
 			(project "Mixer"
 				(path "/322d427a-6aae-4762-92d6-d97688daf29b/8a2849b7-184d-4014-bb98-da9dec8b5f90/2339b41c-0b4b-469c-8280-8e71cc37578f"
-					(reference "R40")
+					(reference "R42")
 					(unit 1)
 				)
@@
 		(in_pos_files yes)
 		(dnp no)
-		(property "Reference" "R46"
+		(property "Reference" "R48"
 			(at 100.33 72.136 90)
 			(show_name no)
@@
 			(project "Mixer"
 				(path "/322d427a-6aae-4762-92d6-d97688daf29b/8a2849b7-184d-4014-bb98-da9dec8b5f90/2339b41c-0b4b-469c-8280-8e71cc37578f"
-					(reference "R46")
+					(reference "R48")
 					(unit 1)
 				)
@@
 		(dnp no)
 		(fields_autoplaced yes)
-		(property "Reference" "U7"
+		(property "Reference" "U9"
 			(at 135.89 48.26 0)
 			(show_name no)
@@
 			(project "Mixer"
 				(path "/322d427a-6aae-4762-92d6-d97688daf29b/8a2849b7-184d-4014-bb98-da9dec8b5f90/2339b41c-0b4b-469c-8280-8e71cc37578f"
-					(reference "U7")
+					(reference "U9")
 					(unit 2)
 				)
@@
 		(dnp no)
 		(fields_autoplaced yes)
-		(property "Reference" "#PWR022"
+		(property "Reference" "#PWR018"
 			(at 82.55 52.07 0)
 			(hide yes)
@@
 			(project "Mixer"
 				(path "/322d427a-6aae-4762-92d6-d97688daf29b/8a2849b7-184d-4014-bb98-da9dec8b5f90/2339b41c-0b4b-469c-8280-8e71cc37578f"
-					(reference "#PWR022")
+					(reference "#PWR018")
 					(unit 1)
 				)
@@
 		(dnp no)
 		(fields_autoplaced yes)
-		(property "Reference" "U6"
+		(property "Reference" "U8"
 			(at 99.06 35.56 0)
 			(show_name no)
@@
 			(project "Mixer"
 				(path "/322d427a-6aae-4762-92d6-d97688daf29b/8a2849b7-184d-4014-bb98-da9dec8b5f90/2339b41c-0b4b-469c-8280-8e71cc37578f"
-					(reference "U6")
+					(reference "U8")
 					(unit 1)
 				)
@@
 		(dnp no)
 		(fields_autoplaced yes)
-		(property "Reference" "#PWR023"
+		(property "Reference" "#PWR019"
 			(at 119.38 52.07 0)
 			(hide yes)
@@
 			(project "Mixer"
 				(path "/322d427a-6aae-4762-92d6-d97688daf29b/8a2849b7-184d-4014-bb98-da9dec8b5f90/2339b41c-0b4b-469c-8280-8e71cc37578f"
-					(reference "#PWR023")
+					(reference "#PWR019")
 					(unit 1)
 				)
@@
 		(in_pos_files yes)
 		(dnp no)
-		(property "Reference" "R52"
+		(property "Reference" "R54"
 			(at 149.352 60.96 90)
 			(show_name no)
@@
 			(project "Mixer"
 				(path "/322d427a-6aae-4762-92d6-d97688daf29b/8a2849b7-184d-4014-bb98-da9dec8b5f90/2339b41c-0b4b-469c-8280-8e71cc37578f"
-					(reference "R52")
+					(reference "R54")
 					(unit 1)
 				)
@@
 		(dnp no)
 		(fields_autoplaced yes)
-		(property "Reference" "U6"
+		(property "Reference" "U8"
 			(at 99.06 48.26 0)
 			(show_name no)
@@
 			(project "Mixer"
 				(path "/322d427a-6aae-4762-92d6-d97688daf29b/8a2849b7-184d-4014-bb98-da9dec8b5f90/2339b41c-0b4b-469c-8280-8e71cc37578f"
-					(reference "U6")
+					(reference "U8")
 					(unit 2)
 				)
@@
 		(dnp no)
 		(fields_autoplaced yes)
-		(property "Reference" "R48"
+		(property "Reference" "R50"
 			(at 121.92 54.61 90)
 			(show_name no)
@@
 			(project "Mixer"
 				(path "/322d427a-6aae-4762-92d6-d97688daf29b/8a2849b7-184d-4014-bb98-da9dec8b5f90/2339b41c-0b4b-469c-8280-8e71cc37578f"
-					(reference "R48")
+					(reference "R50")
 					(unit 1)
 				)
@@
 		(dnp no)
 		(fields_autoplaced yes)
-		(property "Reference" "R49"
+		(property "Reference" "R51"
 			(at 135.89 29.21 90)
 			(show_name no)
@@
 			(project "Mixer"
 				(path "/322d427a-6aae-4762-92d6-d97688daf29b/8a2849b7-184d-4014-bb98-da9dec8b5f90/2339b41c-0b4b-469c-8280-8e71cc37578f"
-					(reference "R49")
-					(unit 1)
-				)
+					(reference "R51")
+					(unit 1)
+				)
