File: KiCAD/Mixer/ch_muteL.kicad_sch (KiCad schematic)
At the start: 9 parts, among them Q2 MMBFJ111, Q3 MMBFJ111, SW1 SW_MEC_5G

Commit message: Rework of schematic, with error fixes and reworked pcb
Parts:
- renumbered C18 to C22, Q2 to Q5, Q3 to Q6, R8 to R64, R9 to R65, R10 to R66, R11 to R67, R12 to R68, SW1 to SW2
Changed lines of the file:
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@@
 		(in_pos_files yes)
 		(dnp no)
-		(property "Reference" "SW1"
+		(property "Reference" "SW2"
 			(at 49.53 66.802 0)
 			(show_name no)
@@
 		(instances
 			(project "Mixer"
-				(path "/322d427a-6aae-4762-92d6-d97688daf29b/8a2849b7-184d-4014-bb98-da9dec8b5f90/bf84a5ed-2042-40b8-aca0-adb831118b62"
-					(reference "SW1")
+				(path "/322d427a-6aae-4762-92d6-d97688daf29b/8a2849b7-184d-4014-bb98-da9dec8b5f90/ec4e71c2-26db-4ba4-aad5-0bfc40b10850"
+					(reference "SW2")
 					(unit 1)
 				)
@@
 		(dnp no)
 		(fields_autoplaced yes)
-		(property "Reference" "R11"
+		(property "Reference" "R67"
 			(at 101.6 55.88 90)
 			(show_name no)
@@
 		(instances
 			(project "Mixer"
-				(path "/322d427a-6aae-4762-92d6-d97688daf29b/8a2849b7-184d-4014-bb98-da9dec8b5f90/bf84a5ed-2042-40b8-aca0-adb831118b62"
-					(reference "R11")
+				(path "/322d427a-6aae-4762-92d6-d97688daf29b/8a2849b7-184d-4014-bb98-da9dec8b5f90/ec4e71c2-26db-4ba4-aad5-0bfc40b10850"
+					(reference "R67")
 					(unit 1)
 				)
@@
 		(dnp no)
 		(fields_autoplaced yes)
-		(property "Reference" "Q3"
+		(property "Reference" "Q6"
 			(at 97.79 69.8499 0)
 			(show_name no)
@@
 		(instances
 			(project "Mixer"
-				(path "/322d427a-6aae-4762-92d6-d97688daf29b/8a2849b7-184d-4014-bb98-da9dec8b5f90/bf84a5ed-2042-40b8-aca0-adb831118b62"
-					(reference "Q3")
+				(path "/322d427a-6aae-4762-92d6-d97688daf29b/8a2849b7-184d-4014-bb98-da9dec8b5f90/ec4e71c2-26db-4ba4-aad5-0bfc40b10850"
+					(reference "Q6")
 					(unit 1)
 				)
@@
 		(dnp no)
 		(fields_autoplaced yes)
-		(property "Reference" "R10"
+		(property "Reference" "R66"
 			(at 62.23 64.77 90)
 			(show_name no)
@@
 		(instances
 			(project "Mixer"
-				(path "/322d427a-6aae-4762-92d6-d97688daf29b/8a2849b7-184d-4014-bb98-da9dec8b5f90/bf84a5ed-2042-40b8-aca0-adb831118b62"
-					(reference "R10")
+				(path "/322d427a-6aae-4762-92d6-d97688daf29b/8a2849b7-184d-4014-bb98-da9dec8b5f90/ec4e71c2-26db-4ba4-aad5-0bfc40b10850"
+					(reference "R66")
 					(unit 1)
 				)
@@
 		(in_pos_files yes)
 		(dnp no)
-		(property "Reference" "C18"
+		(property "Reference" "C22"
 			(at 69.85 82.55 0)
 			(show_name no)
@@
 		(instances
 			(project "Mixer"
-				(path "/322d427a-6aae-4762-92d6-d97688daf29b/8a2849b7-184d-4014-bb98-da9dec8b5f90/bf84a5ed-2042-40b8-aca0-adb831118b62"
-					(reference "C18")
+				(path "/322d427a-6aae-4762-92d6-d97688daf29b/8a2849b7-184d-4014-bb98-da9dec8b5f90/ec4e71c2-26db-4ba4-aad5-0bfc40b10850"
+					(reference "C22")
 					(unit 1)
 				)
@@
 		(dnp no)
 		(fields_autoplaced yes)
-		(property "Reference" "Q2"
+		(property "Reference" "Q5"
 			(at 78.74 69.8499 0)
 			(show_name no)
@@
 		(instances
 			(project "Mixer"
-				(path "/322d427a-6aae-4762-92d6-d97688daf29b/8a2849b7-184d-4014-bb98-da9dec8b5f90/bf84a5ed-2042-40b8-aca0-adb831118b62"
-					(reference "Q2")
+				(path "/322d427a-6aae-4762-92d6-d97688daf29b/8a2849b7-184d-4014-bb98-da9dec8b5f90/ec4e71c2-26db-4ba4-aad5-0bfc40b10850"
+					(reference "Q5")
 					(unit 1)
 				)
@@
 		(in_pos_files yes)
 		(dnp no)
-		(property "Reference" "R12"
+		(property "Reference" "R68"
 			(at 109.22 56.642 90)
 			(show_name no)
@@
 		(instances
 			(project "Mixer"
-				(path "/322d427a-6aae-4762-92d6-d97688daf29b/8a2849b7-184d-4014-bb98-da9dec8b5f90/bf84a5ed-2042-40b8-aca0-adb831118b62"
-					(reference "R12")
+				(path "/322d427a-6aae-4762-92d6-d97688daf29b/8a2849b7-184d-4014-bb98-da9dec8b5f90/ec4e71c2-26db-4ba4-aad5-0bfc40b10850"
+					(reference "R68")
 					(unit 1)
 				)
@@
 		(dnp no)
 		(fields_autoplaced yes)
-		(property "Reference" "R9"
+		(property "Reference" "R65"
 			(at 62.23 55.88 90)
 			(show_name no)
@@
 		(instances
 			(project "Mixer"
-				(path "/322d427a-6aae-4762-92d6-d97688daf29b/8a2849b7-184d-4014-bb98-da9dec8b5f90/bf84a5ed-2042-40b8-aca0-adb831118b62"
-					(reference "R9")
+				(path "/322d427a-6aae-4762-92d6-d97688daf29b/8a2849b7-184d-4014-bb98-da9dec8b5f90/ec4e71c2-26db-4ba4-aad5-0bfc40b10850"
+					(reference "R65")
 					(unit 1)
 				)
@@
 		(dnp no)
 		(fields_autoplaced yes)
-		(property "Reference" "R8"
+		(property "Reference" "R64"
 			(at 58.42 76.1999 0)
 			(show_name no)
@@
 		(instances
 			(project "Mixer"
-				(path "/322d427a-6aae-4762-92d6-d97688daf29b/8a2849b7-184d-4014-bb98-da9dec8b5f90/bf84a5ed-2042-40b8-aca0-adb831118b62"
-					(reference "R8")
-					(unit 1)
-				)
+				(path "/322d427a-6aae-4762-92d6-d97688daf29b/8a2849b7-184d-4014-bb98-da9dec8b5f90/ec4e71c2-26db-4ba4-aad5-0bfc40b10850"
+					(reference "R64")
+					(unit 1)
+				)

Commit message: Final PCB Version that got ordered from JLCPCB
Parts:
- removed C22: 220n, Capacitor_SMD:C_0805_2012Metric_Pad1.18x1.45mm_HandSolder, symbol Device:C
- added C26: 220n, Capacitor_SMD:C_0805_2012Metric_Pad1.18x1.45mm_HandSolder, symbol Device:C
Connections:
- net GND: now also C26.2
- net at Q5.3 (G), Q6.3 (G), R66.2: now also C26.1
